Commit message: implementando o lote B

File: src/aracne_description/urdf/aracne.xacro (robot description, xacro)
@@ -12,6 +12,26 @@
   <xacro:arg name="joint_limits_tibia_lower" default="-2.09"/>
   <xacro:arg name="joint_limits_tibia_upper" default="0.0"/>
+  <ros2_control name="aracne_leg1_controller" type="system">
+    <hardware>
+      <plugin>gz_ros2_control::GazeboSystem</plugin>
+    </hardware>
+    <joint name="leg1_coxa_joint">
+      <command_interface name="position"/>
+      <state_interface name="position"/>
+      <state_interface name="velocity"/>
+    </joint>
+    <joint name="leg1_femur_joint">
+      <command_interface name="position"/>
+      <state_interface name="position"/>
+      <state_interface name="velocity"/>
+    </joint>
+    <joint name="leg1_tibia_joint">
+      <command_interface name="position"/>
+      <state_interface name="position"/>
+      <state_interface name="velocity"/>
+    </joint>
+  </ros2_control>
   <xacro:leg
-    prefix="leg1"
+    leg_prefix="leg1"
     leg_coxa_length="${leg_coxa_length}"
     leg_femur_length="${leg_femur_length}"
@@ -24,3 +44,12 @@
     joint_limits_tibia_upper="${joint_limits_tibia_upper}"
   />
+  <gazebo>
+    <plugin name="gz_ros2_control" filename="libgz_ros2_control_gazebo.so">
+      <ros2_control>
+        <hardware>
+          <plugin>gz_ros2_control::GazeboSystem</plugin>
+        </hardware>
+      </ros2_control>
+    </plugin>
+  </gazebo>
 </robot>

File: src/aracne_description/urdf/leg.xacro (robot description, xacro)
@@ -1,8 +1,8 @@
 <?xml version="1.0"?>
-<xacro:macro name="leg" params="prefix leg_coxa_length leg_femur_length leg_tibia_length joint_limits_coxa_lower joint_limits_coxa_upper joint_limits_femur_lower joint_limits_femur_upper joint_limits_tibia_lower joint_limits_tibia_upper">
+<xacro:macro xmlns:xacro="http://www.ros.org/wiki/xacro" name="leg" params="leg_prefix leg_coxa_length leg_femur_length leg_tibia_length joint_limits_coxa_lower joint_limits_coxa_upper joint_limits_femur_lower joint_limits_femur_upper joint_limits_tibia_lower joint_limits_tibia_upper">
   <xacro:property name="coxa_length" value="${leg_coxa_length}"/>
   <xacro:property name="femur_length" value="${leg_femur_length}"/>
   <xacro:property name="tibia_length" value="${leg_tibia_length}"/>
-  <link name="${prefix}_base_link">
+  <link name="${leg_prefix}_base_link">
     <inertial>
       <mass value="0.1"/>
@@ -22,5 +22,5 @@
     </collision>
   </link>
-  <link name="${prefix}_coxa_link">
+  <link name="${leg_prefix}_coxa_link">
     <inertial>
       <mass value="0.05"/>
@@ -29,5 +29,5 @@
     </inertial>
     <visual>
-      <origin xyz="${coxa_length/2} 0 0" rpy="0 0 0"/>
+      <origin xyz="${coxa_length/2} 0 0" rpy="0 1.5708 0"/>
       <geometry>
         <cylinder length="${coxa_length}" radius="0.01"/>
@@ -36,5 +36,5 @@
     </visual>
     <collision>
-      <origin xyz="${coxa_length/2} 0 0" rpy="0 0 0"/>
+      <origin xyz="${coxa_length/2} 0 0" rpy="0 1.5708 0"/>
       <geometry>
         <cylinder length="${coxa_length}" radius="0.01"/>
@@ -42,12 +42,12 @@
     </collision>
   </link>
-  <joint name="${prefix}_coxa_joint" type="revolute">
-    <parent link="${prefix}_base_link"/>
-    <child link="${prefix}_coxa_link"/>
+  <joint name="${leg_prefix}_coxa_joint" type="revolute">
+    <parent link="${leg_prefix}_base_link"/>
+    <child link="${leg_prefix}_coxa_link"/>
     <origin xyz="0 0 0" rpy="0 0 0"/>
     <axis xyz="0 0 1"/>
     <limit lower="${joint_limits_coxa_lower}" upper="${joint_limits_coxa_upper}" effort="10" velocity="1.0"/>
   </joint>
-  <link name="${prefix}_femur_link">
+  <link name="${leg_prefix}_femur_link">
     <inertial>
       <mass value="0.05"/>
@@ -56,5 +56,5 @@
     </inertial>
     <visual>
-      <origin xyz="0 ${femur_length/2} 0" rpy="0 0 0"/>
+      <origin xyz="0 ${femur_length/2} 0" rpy="1.5708 0 0"/>
       <geometry>
         <cylinder length="${femur_length}" radius="0.01"/>
@@ -63,5 +63,5 @@
     </visual>
     <collision>
-      <origin xyz="0 ${femur_length/2} 0" rpy="0 0 0"/>
+      <origin xyz="0 ${femur_length/2} 0" rpy="1.5708 0 0"/>
       <geometry>
         <cylinder length="${femur_length}" radius="0.01"/>
@@ -69,12 +69,12 @@
     </collision>
   </link>
-  <joint name="${prefix}_femur_joint" type="revolute">
-    <parent link="${prefix}_coxa_link"/>
-    <child link="${prefix}_femur_link"/>
+  <joint name="${leg_prefix}_femur_joint" type="revolute">
+    <parent link="${leg_prefix}_coxa_link"/>
+    <child link="${leg_prefix}_femur_link"/>
     <origin xyz="${coxa_length} 0 0" rpy="0 0 0"/>
     <axis xyz="0 1 0"/>
     <limit lower="${joint_limits_femur_lower}" upper="${joint_limits_femur_upper}" effort="10" velocity="1.0"/>
   </joint>
-  <link name="${prefix}_tibia_link">
+  <link name="${leg_prefix}_tibia_link">
     <inertial>
       <mass value="0.05"/>
@@ -83,5 +83,5 @@
     </inertial>
     <visual>
-      <origin xyz="0 ${tibia_length/2} 0" rpy="0 0 0"/>
+      <origin xyz="0 ${tibia_length/2} 0" rpy="1.5708 0 0"/>
       <geometry>
         <cylinder length="${tibia_length}" radius="0.01"/>
@@ -90,5 +90,5 @@
     </visual>
     <collision>
-      <origin xyz="0 ${tibia_length/2} 0" rpy="0 0 0"/>
+      <origin xyz="0 ${tibia_length/2} 0" rpy="1.5708 0 0"/>
       <geometry>
         <cylinder length="${tibia_length}" radius="0.01"/>
@@ -96,19 +96,10 @@
     </collision>
   </link>
-  <joint name="${prefix}_tibia_joint" type="revolute">
-    <parent link="${prefix}_femur_link"/>
-    <child link="${prefix}_tibia_link"/>
+  <joint name="${leg_prefix}_tibia_joint" type="revolute">
+    <parent link="${leg_prefix}_femur_link"/>
+    <child link="${leg_prefix}_tibia_link"/>
     <origin xyz="0 ${femur_length} 0" rpy="0 0 0"/>
     <axis xyz="0 1 0"/>
     <limit lower="${joint_limits_tibia_lower}" upper="${joint_limits_tibia_upper}" effort="10" velocity="1.0"/>
   </joint>
-  <gazebo>
-    <plugin name="gz_ros2_control" filename="libgz_ros2_control_gazebo.so">
-      <ros2_control>
-        <hardware>
-          <plugin>gz_ros2_control::GazeboSystem</plugin>
-        </hardware>
-      </ros2_control>
-    </plugin>
-  </gazebo>
 </xacro:macro>

Commit message: git commit -m "fix(mark1): finalize Lote B.1 Xacro and gz_ros2_control integration" \   -m "Fix Xacro macro inclusion and argument forwarding, remove duplicate ros2_control configuration, align gz_ros2_control plugins with ROS 2 Jazzy/Gazebo Harmonic, and validate with xacro, check_urdf and colcon build."

File: src/aracne_description/urdf/aracne.xacro (robot description, xacro)
@@ -12,7 +12,7 @@
   <xacro:arg name="joint_limits_tibia_lower" default="-2.09"/>
   <xacro:arg name="joint_limits_tibia_upper" default="0.0"/>
-  <ros2_control name="aracne_leg1_controller" type="system">
+    <ros2_control name="aracne_leg1_controller" type="system">
     <hardware>
-      <plugin>gz_ros2_control::GazeboSystem</plugin>
+      <plugin>gz_ros2_control/GazeboSimSystem</plugin>
     </hardware>
     <joint name="leg1_coxa_joint">
@@ -32,23 +32,20 @@
     </joint>
   </ros2_control>
-  <xacro:leg
+    <xacro:leg
     leg_prefix="leg1"
-    leg_coxa_length="${leg_coxa_length}"
-    leg_femur_length="${leg_femur_length}"
-    leg_tibia_length="${leg_tibia_length}"
-    joint_limits_coxa_lower="${joint_limits_coxa_lower}"
-    joint_limits_coxa_upper="${joint_limits_coxa_upper}"
-    joint_limits_femur_lower="${joint_limits_femur_lower}"
-    joint_limits_femur_upper="${joint_limits_femur_upper}"
-    joint_limits_tibia_lower="${joint_limits_tibia_lower}"
-    joint_limits_tibia_upper="${joint_limits_tibia_upper}"
+    leg_coxa_length="$(arg leg_coxa_length)"
+    leg_femur_length="$(arg leg_femur_length)"
+    leg_tibia_length="$(arg leg_tibia_length)"
+    joint_limits_coxa_lower="$(arg joint_limits_coxa_lower)"
+    joint_limits_coxa_upper="$(arg joint_limits_coxa_upper)"
+    joint_limits_femur_lower="$(arg joint_limits_femur_lower)"
+    joint_limits_femur_upper="$(arg joint_limits_femur_upper)"
+    joint_limits_tibia_lower="$(arg joint_limits_tibia_lower)"
+    joint_limits_tibia_upper="$(arg joint_limits_tibia_upper)"
   />
-  <gazebo>
-    <plugin name="gz_ros2_control" filename="libgz_ros2_control_gazebo.so">
-      <ros2_control>
-        <hardware>
-          <plugin>gz_ros2_control::GazeboSystem</plugin>
-        </hardware>
-      </ros2_control>
+      <gazebo>
+    <plugin
+      filename="libgz_ros2_control-system.so"
+      name="gz_ros2_control::GazeboSimROS2ControlPlugin">
     </plugin>
   </gazebo>

File: src/aracne_description/urdf/leg.xacro (robot description, xacro)
@@ -1,4 +1,5 @@
 <?xml version="1.0"?>
-<xacro:macro xmlns:xacro="http://www.ros.org/wiki/xacro" name="leg" params="leg_prefix leg_coxa_length leg_femur_length leg_tibia_length joint_limits_coxa_lower joint_limits_coxa_upper joint_limits_femur_lower joint_limits_femur_upper joint_limits_tibia_lower joint_limits_tibia_upper">
+<robot xmlns:xacro="http://www.ros.org/wiki/xacro">
+  <xacro:macro name="leg" params="leg_prefix leg_coxa_length leg_femur_length leg_tibia_length joint_limits_coxa_lower joint_limits_coxa_upper joint_limits_femur_lower joint_limits_femur_upper joint_limits_tibia_lower joint_limits_tibia_upper">
   <xacro:property name="coxa_length" value="${leg_coxa_length}"/>
   <xacro:property name="femur_length" value="${leg_femur_length}"/>
@@ -102,4 +103,5 @@
     <axis xyz="0 1 0"/>
     <limit lower="${joint_limits_tibia_lower}" upper="${joint_limits_tibia_upper}" effort="10" velocity="1.0"/>
-  </joint>
+    </joint>
 </xacro:macro>
+</robot>
